File: circuits/inverter/drivers.sch (KiCad schematic (older format))
At the start: 0 parts

Commit message: bulk-updates libraries and schematics
schematic is updated to Kicad 5.1.14
updates various sheets with new circuits
adds various component libraries
Parts:
- added U? (x2): Si8715BC-A-IS, symbol Si871x_2x:Si8715BC-A-IS
Changed lines of the file:
@@
-EESchema Schematic File Version 2
-LIBS:lm317
-LIBS:kv30f
-LIBS:OSSI_standard_components
-LIBS:connectors
-LIBS:lm4030
-LIBS:acs722
+EESchema Schematic File Version 4
 LIBS:OSSI_MK_I-cache
-EELAYER 25 0
+EELAYER 30 0
 EELAYER END
 $Descr A4 11693 8268
 encoding utf-8
-Sheet 7 11
+Sheet 10 11
 Title ""
 Date ""
@@
 Comment4 ""
 $EndDescr
+Text HLabel 1200 1700 0    50   Input ~ 0
+T1_IN
+Text HLabel 1225 2250 0    50   Input ~ 0
+T2_IN
+Text HLabel 1200 2950 0    50   Input ~ 0
+T3_IN
+Text HLabel 1250 3525 0    50   Input ~ 0
+T4_IN
+Text HLabel 9900 1600 2    50   Output ~ 0
+T1_OUT
+Text HLabel 9900 1925 2    50   Output ~ 0
+T2_OUT
+Text HLabel 9875 2225 2    50   Output ~ 0
+T3_OUT
+Text HLabel 9875 2625 2    50   Output ~ 0
+T4_OUT
+$Comp
+L Si871x_2x:Si8715BC-A-IS U?
+U 1 1 5D6A8098
+P 3450 1225
+F 0 "U?" H 3450 975 39  0000 C CNN
+F 1 "Si8715BC-A-IS" H 3450 1475 50  0000 C CNN
+F 2 "" H 3450 925 39  0001 C CNN
+F 3 "" H 3450 1550 50  0000 C CNN
+	1    3450 1225
+	1    0    0    -1
+$EndComp
+$Comp
+L Si871x_2x:Si8715BC-A-IS U?
+U 1 1 5D6A9B2E
+P 3450 1950
+F 0 "U?" H 3450 1700 39  0000 C CNN
+F 1 "Si8715BC-A-IS" H 3450 2200 50  0000 C CNN
+F 2 "" H 3450 1650 39  0001 C CNN
+F 3 "" H 3350 1950 50  0000 C CNN
+	1    3450 1950
+	1    0    0    -1
+$EndComp
 $EndSCHEMATC
