File: circuits/inverter/DC_booster.kicad_sch (KiCad schematic)
At the start: 31 parts

Commit message: converts libraries to Kicad 6 format, updates bridge driver
Parts:
- gave numbers to parts that had none: 5
Changed lines of the file:
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@@
   (symbol (lib_id "OSSI_standard_components:Resistor") (at 78.74 40.64 0) (unit 1)
     (in_bom yes) (on_board yes)
-    (property "Reference" "" (id 0) (at 78.74 42.672 0)
+    (property "Reference" "R?" (id 0) (at 78.74 42.672 0)
       (effects (font (size 0.9906 0.9906)))
     )
@@
   (symbol (lib_id "OSSI_standard_components:Resistor") (at 102.87 55.88 0) (unit 1)
     (in_bom yes) (on_board yes)
-    (property "Reference" "" (id 0) (at 102.87 57.912 0)
+    (property "Reference" "R?" (id 0) (at 102.87 57.912 0)
       (effects (font (size 0.9906 0.9906)))
     )
@@
   (symbol (lib_id "OSSI_standard_components:Resistor") (at 111.76 48.26 90) (mirror x) (unit 1)
     (in_bom yes) (on_board yes)
-    (property "Reference" "" (id 0) (at 113.792 48.26 0)
+    (property "Reference" "R?" (id 0) (at 113.792 48.26 0)
       (effects (font (size 0.9906 0.9906)))
     )
@@
   (symbol (lib_id "OSSI_standard_components:Capacitor") (at 123.19 45.72 0) (unit 1)
     (in_bom yes) (on_board yes)
-    (property "Reference" "" (id 0) (at 124.714 48.26 0)
+    (property "Reference" "C?" (id 0) (at 124.714 48.26 0)
       (effects (font (size 0.9906 0.9906)) (justify left))
     )
@@
   (symbol (lib_id "OSSI_standard_components:PMOS") (at 138.43 53.34 0) (unit 1)
     (in_bom yes) (on_board yes)
-    (property "Reference" "" (id 0) (at 138.43 58.42 0)
+    (property "Reference" "Q?" (id 0) (at 138.43 58.42 0)
       (effects (font (size 0.9906 0.9906)) (justify right))
     )
@@
   (symbol (lib_id "OSSI_standard_components:Capacitor") (at 102.87 64.77 90) (mirror x) (unit 1)
     (in_bom yes) (on_board yes)
-    (property "Reference" "" (id 0) (at 104.14 67.31 90)
+    (property "Reference" "C?" (id 0) (at 104.14 67.31 90)
       (effects (font (size 0.9906 0.9906)) (justify right))
     )
@@
   (symbol (lib_id "OSSI_standard_components:NMOS") (at 87.63 60.96 0) (unit 1)
     (in_bom yes) (on_board yes)
-    (property "Reference" "" (id 0) (at 87.63 66.04 0)
+    (property "Reference" "Q?" (id 0) (at 87.63 66.04 0)
       (effects (font (size 0.9906 0.9906)) (justify right))
     )
@@
   (symbol (lib_id "OSSI_standard_components:Capacitor") (at 78.74 69.85 0) (unit 1)
     (in_bom yes) (on_board yes)
-    (property "Reference" "" (id 0) (at 80.264 72.39 0)
+    (property "Reference" "C?" (id 0) (at 80.264 72.39 0)
       (effects (font (size 0.9906 0.9906)) (justify left))
     )
@@
   (symbol (lib_id "OSSI_standard_components:Resistor") (at 63.5 72.39 0) (unit 1)
     (in_bom yes) (on_board yes)
-    (property "Reference" "" (id 0) (at 63.5 74.422 0)
+    (property "Reference" "R?" (id 0) (at 63.5 74.422 0)
       (effects (font (size 0.9906 0.9906)))
     )
@@
   (symbol (lib_id "OSSI_standard_components:Schottky") (at 63.5 63.5 0) (mirror y) (unit 1)
     (in_bom yes) (on_board yes)
-    (property "Reference" "" (id 0) (at 63.5 66.04 0)
+    (property "Reference" "D?" (id 0) (at 63.5 66.04 0)
       (effects (font (size 0.9906 0.9906)))
     )
@@
   (symbol (lib_id "OSSI_standard_components:Schottky") (at 63.5 88.9 0) (unit 1)
     (in_bom yes) (on_board yes)
-    (property "Reference" "" (id 0) (at 63.5 91.44 0)
+    (property "Reference" "D?" (id 0) (at 63.5 91.44 0)
       (effects (font (size 0.9906 0.9906)))
     )
@@
   (symbol (lib_id "OSSI_standard_components:Resistor") (at 63.5 97.79 0) (unit 1)
     (in_bom yes) (on_board yes)
-    (property "Reference" "" (id 0) (at 63.5 99.822 0)
+    (property "Reference" "R?" (id 0) (at 63.5 99.822 0)
       (effects (font (size 0.9906 0.9906)))
     )
@@
   (symbol (lib_id "OSSI_standard_components:Capacitor") (at 78.74 105.41 0) (unit 1)
     (in_bom yes) (on_board yes)
-    (property "Reference" "" (id 0) (at 80.264 107.95 0)
+    (property "Reference" "C?" (id 0) (at 80.264 107.95 0)
       (effects (font (size 0.9906 0.9906)) (justify left))
     )
@@
   (symbol (lib_id "OSSI_standard_components:PMOS") (at 87.63 95.25 0) (unit 1)
     (in_bom yes) (on_board yes)
-    (property "Reference" "" (id 0) (at 87.63 100.33 0)
+    (property "Reference" "Q?" (id 0) (at 87.63 100.33 0)
       (effects (font (size 0.9906 0.9906)) (justify right))
     )
@@
   (symbol (lib_id "OSSI_standard_components:Capacitor") (at 102.87 93.98 90) (mirror x) (unit 1)
     (in_bom yes) (on_board yes)
-    (property "Reference" "" (id 0) (at 104.14 96.52 90)
+    (property "Reference" "C?" (id 0) (at 104.14 96.52 90)
       (effects (font (size 0.9906 0.9906)) (justify right))
     )
@@
   (symbol (lib_id "OSSI_standard_components:Resistor") (at 102.87 101.6 0) (unit 1)
     (in_bom yes) (on_board yes)
-    (property "Reference" "" (id 0) (at 102.87 103.632 0)
+    (property "Reference" "R?" (id 0) (at 102.87 103.632 0)
       (effects (font (size 0.9906 0.9906)))
     )
@@
   (symbol (lib_id "OSSI_standard_components:NMOS") (at 111.76 115.57 0) (unit 1)
     (in_bom yes) (on_board yes)
-    (property "Reference" "" (id 0) (at 111.76 120.65 0)
+    (property "Reference" "Q?" (id 0) (at 111.76 120.65 0)
       (effects (font (size 0.9906 0.9906)) (justify right))
     )
@@
   (symbol (lib_id "OSSI_standard_components:Resistor") (at 129.54 113.03 90) (mirror x) (unit 1)
     (in_bom yes) (on_board yes)
-    (property "Reference" "" (id 0) (at 131.572 113.03 0)
+    (property "Reference" "R?" (id 0) (at 131.572 113.03 0)
       (effects (font (size 0.9906 0.9906)))
     )
@@
   (symbol (lib_id "OSSI_standard_components:NMOS") (at 138.43 99.06 0) (unit 1)
     (in_bom yes) (on_board yes)
-    (property "Reference" "" (id 0) (at 138.43 104.14 0)
+    (property "Reference" "Q?" (id 0) (at 138.43 104.14 0)
       (effects (font (size 0.9906 0.9906)) (justify right))
     )
@@
   (symbol (lib_id "OSSI_standard_components:Resistor") (at 156.21 80.01 0) (unit 1)
     (in_bom yes) (on_board yes)
-    (property "Reference" "" (id 0) (at 156.21 82.042 0)
+    (property "Reference" "R?" (id 0) (at 156.21 82.042 0)
       (effects (font (size 0.9906 0.9906)))
     )
@@
   (symbol (lib_id "OSSI_standard_components:Capacitor") (at 185.42 88.9 0) (unit 1)
     (in_bom yes) (on_board yes)
-    (property "Reference" "" (id 0) (at 186.944 91.44 0)
+    (property "Reference" "C?" (id 0) (at 186.944 91.44 0)
       (effects (font (size 0.9906 0.9906)) (justify left))
     )
@@
   (symbol (lib_id "OSSI_standard_components:Resistor") (at 185.42 77.47 90) (mirror x) (unit 1)
     (in_bom yes) (on_board yes)
-    (property "Reference" "" (id 0) (at 187.452 77.47 0)
+    (property "Reference" "R?" (id 0) (at 187.452 77.47 0)
       (effects (font (size 0.9906 0.9906)))
     )
@@
   (symbol (lib_id "OSSI_standard_components:IGBT") (at 172.72 77.47 0) (unit 1)
     (in_bom yes) (on_board yes)
-    (property "Reference" "" (id 0) (at 172.72 82.55 0)
+    (property "Reference" "Q?" (id 0) (at 172.72 82.55 0)
       (effects (font (size 0.9906 0.9906)) (justify right))
     )
@@
   (symbol (lib_id "OSSI_standard_components:Diode") (at 215.9 26.67 0) (unit 1)
     (in_bom yes) (on_board yes)
-    (property "Reference" "" (id 0) (at 215.9 29.21 0)
+    (property "Reference" "D?" (id 0) (at 215.9 29.21 0)
       (effects (font (size 0.9906 0.9906)))
     )
@@
   (symbol (lib_id "OSSI_standard_components:Resistor") (at 209.55 19.05 0) (unit 1)
     (in_bom yes) (on_board yes)
-    (property "Reference" "" (id 0) (at 209.55 21.082 0)
+    (property "Reference" "R?" (id 0) (at 209.55 21.082 0)
       (effects (font (size 0.9906 0.9906)))
     )
@@
   (symbol (lib_id "OSSI_standard_components:Capacitor") (at 224.79 19.05 90) (mirror x) (unit 1)
     (in_bom yes) (on_board yes)
-    (property "Reference" "" (id 0) (at 226.06 21.59 90)
+    (property "Reference" "C?" (id 0) (at 226.06 21.59 90)
       (effects (font (size 0.9906 0.9906)) (justify right))
     )
@@
   (symbol (lib_id "OSSI_standard_components:Capacitor_pol") (at 233.68 58.42 0) (unit 1)
     (in_bom yes) (on_board yes)
-    (property "Reference" "" (id 0) (at 234.823 60.96 0)
+    (property "Reference" "C?" (id 0) (at 234.823 60.96 0)
       (effects (font (size 0.9906 0.9906)) (justify left))
     )
@@
   (symbol (lib_id "OSSI_standard_components:Capacitor_pol") (at 245.11 58.42 0) (unit 1)
     (in_bom yes) (on_board yes)
-    (property "Reference" "" (id 0) (at 246.253 60.96 0)
+    (property "Reference" "C?" (id 0) (at 246.253 60.96 0)
       (effects (font (size 0.9906 0.9906)) (justify left))
     )
@@
   (symbol (lib_id "OSSI_standard_components:Capacitor_pol") (at 256.54 58.42 0) (unit 1)
     (in_bom yes) (on_board yes)
-    (property "Reference" "" (id 0) (at 257.683 60.96 0)
+    (property "Reference" "C?" (id 0) (at 257.683 60.96 0)
       (effects (font (size 0.9906 0.9906)) (justify left))
     )
@@
   (symbol (lib_id "OSSI_standard_components:Resistor") (at 46.99 90.17 90) (mirror x) (unit 1)
     (in_bom yes) (on_board yes)
-    (property "Reference" "" (id 0) (at 49.022 90.17 0)
+    (property "Reference" "R?" (id 0) (at 49.022 90.17 0)
       (effects (font (size 0.9906 0.9906)))
     )
@@
   (symbol (lib_id "OSSI_standard_components:Inductor") (at 136.525 26.67 0) (unit 1)
     (in_bom yes) (on_board yes)
-    (property "Reference" "" (id 0) (at 136.525 27.94 0)
-      (effects (font (size 0.9906 0.9906)))
-    )
+    (property "Reference" "L?" (id 0) (at 136.525 27.94 0)
+      (effects (font (size 0.9906 0.9906)))
+    )
