File: circuits/OSSI_CM2/OSSI_CM2.kicad_pcb (KiCad board)
At the start: 4 copper layers, 49.5 x 54.9 mm, 76 parts, among them U101 STM32L412C8T6, U103 LM75B, U104 OPA2317, X101 PINHEADER_2×5, X201 Conn_01x20_Pin, X202 Conn_01x21_Pin, Y101 10MHz

Commit message: updates PCB with pinout comments, adds pinout PDF
Other:
- board text added: "(Boost_T1) PB10"
- board text added: "(Bridge_T1) PA8"
- board text added: "(Bridge_T2) PA9"
- board text added: "(Bridge_T3) PA10"
- board text added: "(Bridge_T4) PA11"
- board text added: "(Grid_Relay_Ctrl) PB8"
- board text added: "(HISIDE_PWM_µC) PB3"
- board text added: "(I2C_Clk) PB13"
- board text added: "(I2C_Dat) PB14"
- board text added: "(Inv_Relay_Ctrl) PB5"
- board text added: "(LED gn) PA12"
- board text added: "(LED rd) PA15"
- board text added: "(Relay_Voltage_Ctrl) PB11"
- board text added: "(UART_RX) PB7"
- board text added: "(UART_TX) PB6"
- board text added: "+1V25_REF"
- board text added: "+2V50_REF"
- board text added: "+3V3"
- board text added: "+3V3_ANA"
- board text added: "AGND"
- board text added: "GND"
- board text added: "PA1/ADC1_6 (AC_Grid_Voltage)"
- board text added: "PA2/ADC12_7 (Relay_Ctrl_Voltage)"
- board text added: "PA3/ADC12_8 (DC_Link_Voltage)"
- board text added: "PA4/ADC12_9 (AC_Current)"
- board text added: "PA5/ADC12_10 (AC_Relay_Voltage)"
- board text added: "PA6/ADC12_11 (DC_Input_Voltage)"
- board text added: "PA7/ADC12_12 (DC_Current)"
- board text added: "PB0/ADC12_15 (AC_Inverter_Voltage)"
- board text added: "PB1 (LED_Red_Ctrl)"
- board text added: "PB4 (LED_Green_Ctrl)"
Changed lines of the file:
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@@
     (pad_to_mask_clearance 0)
     (pcbplotparams
-      (layerselection 0x00010fc_ffffffff)
-      (plot_on_all_layers_selection 0x0000000_00000000)
+      (layerselection 0x0000000_7ffffff9)
+      (plot_on_all_layers_selection 0x0001220_00000001)
       (disableapertmacros false)
       (usegerberextensions false)
@@
       (sketchpadsonfab false)
       (subtractmaskfromsilk false)
-      (outputformat 1)
+      (outputformat 4)
       (mirror false)
       (drillshape 0)
       (scaleselection 1)
-      (outputdirectory "fabrication")
+      (outputdirectory "bom/")
     )
   )
@@
     (effects (font (size 1.2 1.2) (thickness 0.3) bold) (justify bottom))
   )
+  (gr_text "AGND" (at 112.519048 101) (layer "Cmts.User")
+    (effects (font (size 1 1) (thickness 0.154)) (justify left bottom))
+  )
+  (gr_text "+3V3\n" (at 116.6 126.4) (layer "Cmts.User")
+    (effects (font (size 1 1) (thickness 0.154)) (justify right bottom))
+  )
+  (gr_text "(LED rd) PA15" (at 150.1 72.1 90) (layer "Cmts.User")
+    (effects (font (size 1 1) (thickness 0.154)) (justify left bottom))
+  )
+  (gr_text "GND" (at 113.376191 123.8) (layer "Cmts.User")
+    (effects (font (size 1 1) (thickness 0.154)) (justify left bottom))
+  )
+  (gr_text "+2V50_REF\n" (at 107.947619 83.1) (layer "Cmts.User")
+    (effects (font (size 1 1) (thickness 0.154)) (justify left bottom))
+  )
+  (gr_text "PB4 (LED_Green_Ctrl)" (at 116.8 121.2) (layer "Cmts.User")
+    (effects (font (size 1 1) (thickness 0.154)) (justify right bottom))
+  )
+  (gr_text "(Grid_Relay_Ctrl) PB8" (at 167.6 78) (layer "Cmts.User")
+    (effects (font (size 1 1) (thickness 0.154)) (justify left bottom))
+  )
+  (gr_text " PA6/ADC12_11 (DC_Input_Voltage)" (at 116.8 105.9) (layer "Cmts.User")
+    (effects (font (size 1 1) (thickness 0.154)) (justify right bottom))
+  )
+  (gr_text "AGND" (at 112.519048 108.5) (layer "Cmts.User")
+    (effects (font (size 1 1) (thickness 0.154)) (justify left bottom))
+  )
+  (gr_text "+1V25_REF\n" (at 107.947619 80.7) (layer "Cmts.User")
+    (effects (font (size 1 1) (thickness 0.154)) (justify left bottom))
+  )
+  (gr_text "(Relay_Voltage_Ctrl) PB11" (at 167.7 100.9) (layer "Cmts.User")
+    (effects (font (size 1 1) (thickness 0.154)) (justify left bottom))
+  )
+  (gr_text "PA7/ADC12_12 (DC_Current)" (at 116.8 111) (layer "Cmts.User")
+    (effects (font (size 1 1) (thickness 0.154)) (justify right bottom))
+  )
+  (gr_text "(I2C_Dat) PB14" (at 167.6 116.1) (layer "Cmts.User")
+    (effects (font (size 1 1) (thickness 0.154)) (justify left bottom))
+  )
+  (gr_text "PA1/ADC1_6 (AC_Grid_Voltage)" (at 116.7 88) (layer "Cmts.User")
+    (effects (font (size 1 1) (thickness 0.154)) (justify right bottom))
+  )
+  (gr_text "(Boost_T1) PB10" (at 167.6 105.9) (layer "Cmts.User")
+    (effects (font (size 1 1) (thickness 0.154)) (justify left bottom))
+  )
+  (gr_text "(Bridge_T3) PA10" (at 167.6 90.7) (layer "Cmts.User")
+    (effects (font (size 1 1) (thickness 0.154)) (justify left bottom))
+  )
+  (gr_text "PA3/ADC12_8 (DC_Link_Voltage)" (at 116.7 95.8) (layer "Cmts.User")
+    (effects (font (size 1 1) (thickness 0.154)) (justify right bottom))
+  )
+  (gr_text "PA4/ADC12_9 (AC_Current)" (at 116.7 98.3) (layer "Cmts.User")
+    (effects (font (size 1 1) (thickness 0.154)) (justify right bottom))
+  )
+  (gr_text "(HISIDE_PWM_µC) PB3" (at 167.6 108.5) (layer "Cmts.User")
+    (effects (font (size 1 1) (thickness 0.154)) (justify left bottom))
+  )
+  (gr_text "GND" (at 167.6 88.1) (layer "Cmts.User")
+    (effects (font (size 1 1) (thickness 0.154)) (justify left bottom))
+  )
+  (gr_text "(UART_TX) PB6" (at 167.6 121.2) (layer "Cmts.User")
+    (effects (font (size 1 1) (thickness 0.154)) (justify left bottom))
+  )
+  (gr_text "(LED gn) PA12" (at 154 72.1 90) (layer "Cmts.User")
+    (effects (font (size 1 1) (thickness 0.154)) (justify left bottom))
+  )
+  (gr_text "+3V3_ANA\n" (at 108.9 78.2) (layer "Cmts.User")
+    (effects (font (size 1 1) (thickness 0.154)) (justify left bottom))
+  )
+  (gr_text "GND" (at 167.6 103.4) (layer "Cmts.User")
+    (effects (font (size 1 1) (thickness 0.154)) (justify left bottom))
+  )
+  (gr_text "(Bridge_T4) PA11" (at 167.7 85.6) (layer "Cmts.User")
+    (effects (font (size 1 1) (thickness 0.154)) (justify left bottom))
+  )
+  (gr_text "GND" (at 167.6 118.6) (layer "Cmts.User")
+    (effects (font (size 1 1) (thickness 0.154)) (justify left bottom))
+  )
+  (gr_text "(Bridge_T1) PA8" (at 167.6 98.4) (layer "Cmts.User")
+    (effects (font (size 1 1) (thickness 0.154)) (justify left bottom))
+  )
+  (gr_text "(Bridge_T2) PA9" (at 167.6 93.3) (layer "Cmts.User")
+    (effects (font (size 1 1) (thickness 0.154)) (justify left bottom))
+  )
+  (gr_text "PB0/ADC12_15 (AC_Inverter_Voltage)" (at 116.8 113.6) (layer "Cmts.User")
+    (effects (font (size 1 1) (thickness 0.154)) (justify right bottom))
+  )
+  (gr_text "GND" (at 167.6 75.4) (layer "Cmts.User")
+    (effects (font (size 1 1) (thickness 0.154)) (justify left bottom))
+  )
+  (gr_text "PB1 (LED_Red_Ctrl)" (at 116.8 118.7) (layer "Cmts.User")
+    (effects (font (size 1 1) (thickness 0.154)) (justify right bottom))
+  )
+  (gr_text "AGND" (at 112.519048 85.7) (layer "Cmts.User")
+    (effects (font (size 1 1) (thickness 0.154)) (justify left bottom))
+  )
+  (gr_text "PA2/ADC12_7 (Relay_Ctrl_Voltage)" (at 116.7 90.8) (layer "Cmts.User")
+    (effects (font (size 1 1) (thickness 0.154)) (justify right bottom))
+  )
+  (gr_text "(I2C_Clk) PB13" (at 167.6 113.6) (layer "Cmts.User")
+    (effects (font (size 1 1) (thickness 0.154)) (justify left bottom))
+  )
+  (gr_text "AGND" (at 112.519048 116.2) (layer "Cmts.User")
+    (effects (font (size 1 1) (thickness 0.154)) (justify left bottom))
+  )
+  (gr_text "(UART_RX) PB7" (at 167.6 123.8) (layer "Cmts.User")
+    (effects (font (size 1 1) (thickness 0.154)) (justify left bottom))
+  )
+  (gr_text "GND" (at 167.6 110.9) (layer "Cmts.User")
+    (effects (font (size 1 1) (thickness 0.154)) (justify left bottom))
+  )
+  (gr_text "GND" (at 167.6 95.7) (layer "Cmts.User")
+    (effects (font (size 1 1) (thickness 0.154)) (justify left bottom))
+  )
+  (gr_text "GND" (at 167.6 80.5) (layer "Cmts.User")
+    (effects (font (size 1 1) (thickness 0.154)) (justify left bottom))
+  )
+  (gr_text "PA5/ADC12_10 (AC_Relay_Voltage)" (at 116.8 103.4) (layer "Cmts.User")
+    (effects (font (size 1 1) (thickness 0.154)) (justify right bottom))
+  )
+  (gr_text "(Inv_Relay_Ctrl) PB5" (at 167.7 83.1) (layer "Cmts.User")
+    (effects (font (size 1 1) (thickness 0.154)) (justify left bottom))
+  )
+  (gr_text "GND" (at 167.6 126.2) (layer "Cmts.User")
+    (effects (font (size 1 1) (thickness 0.154)) (justify left bottom))
+  )
+  (gr_text "AGND" (at 112.519048 93.2) (layer "Cmts.User")
+    (effects (font (size 1 1) (thickness 0.154)) (justify left bottom))
+  )
   (dimension (type aligned) (layer "Dwgs.User")
     (pts (xy 119.38 129.54) (xy 165.1 129.54))
@@
   )
   (dimension (type aligned) (layer "Dwgs.User")
-    (pts (xy 166.488 73.286) (xy 166.488 128.15))
+    (pts (xy 186.288 73.286) (xy 186.288 128.15))
     (height -4.012)
-    (gr_text "54.8640 mm" (at 169.346 100.718 90) (layer "Dwgs.User")
+    (gr_text "54.8640 mm" (at 189.146 100.718 90) (layer "Dwgs.User")
       (effects (font (size 1 1) (thickness 0.154)))
     )

Commit message: adds pin description for debug port
Other:
- board text added: "BOOT0"
- board text added: "SCLK"
- board text added: "SDIO"
- board text added: "SWO"
- board text added: "~{RESET}"
Changed lines of the file:
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@@
+    (effects (font (size 1 1) (thickness 0.154)) (justify right bottom))
+  )
+  (gr_text "SCLK" (at 136.2 129.1 45) (layer "Cmts.User")
     (effects (font (size 1 1) (thickness 0.154)) (justify right bottom))
   )
@@
   (gr_text "+2V50_REF\n" (at 107.947619 83.1) (layer "Cmts.User")
     (effects (font (size 1 1) (thickness 0.154)) (justify left bottom))
+  )
+  (gr_text "~{RESET}" (at 144.1 129.3 45) (layer "Cmts.User")
+    (effects (font (size 1 1) (thickness 0.154)) (justify right bottom))
   )
   (gr_text "PB4 (LED_Green_Ctrl)" (at 116.8 121.2) (layer "Cmts.User")
@@
     (effects (font (size 1 1) (thickness 0.154)) (justify left bottom))
   )
+  (gr_text "SDIO" (at 133.5 129 45) (layer "Cmts.User")
+    (effects (font (size 1 1) (thickness 0.154)) (justify right bottom))
+  )
   (gr_text "+1V25_REF\n" (at 107.947619 80.7) (layer "Cmts.User")
     (effects (font (size 1 1) (thickness 0.154)) (justify left bottom))
@@
   (gr_text "(Relay_Voltage_Ctrl) PB11" (at 167.7 100.9) (layer "Cmts.User")
     (effects (font (size 1 1) (thickness 0.154)) (justify left bottom))
+  )
+  (gr_text "+3V3\n" (at 133.3 132.7 45) (layer "Cmts.User")
+    (effects (font (size 1 1) (thickness 0.154)) (justify right bottom))
   )
   (gr_text "PA7/ADC12_12 (DC_Current)" (at 116.8 111) (layer "Cmts.User")
@@
     (effects (font (size 1 1) (thickness 0.154)) (justify left bottom))
   )
+  (gr_text "GND" (at 136.4 135.3 45) (layer "Cmts.User")
+    (effects (font (size 1 1) (thickness 0.154)) (justify left bottom))
+  )
   (gr_text "(Bridge_T2) PA9" (at 167.6 93.3) (layer "Cmts.User")
     (effects (font (size 1 1) (thickness 0.154)) (justify left bottom))
@@
     (effects (font (size 1 1) (thickness 0.154)) (justify left bottom))
   )
+  (gr_text "SWO" (at 138.6 129 45) (layer "Cmts.User")
+    (effects (font (size 1 1) (thickness 0.154)) (justify right bottom))
+  )
+  (gr_text "GND" (at 133.8 135.3 45) (layer "Cmts.User")
+    (effects (font (size 1 1) (thickness 0.154)) (justify left bottom))
+  )
   (gr_text "GND" (at 167.6 110.9) (layer "Cmts.User")
     (effects (font (size 1 1) (thickness 0.154)) (justify left bottom))
   )
   (gr_text "GND" (at 167.6 95.7) (layer "Cmts.User")
+    (effects (font (size 1 1) (thickness 0.154)) (justify left bottom))
+  )
+  (gr_text "BOOT0" (at 141.5 128.9 45) (layer "Cmts.User")
+    (effects (font (size 1 1) (thickness 0.154)) (justify right bottom))
+  )
+  (gr_text "GND" (at 141.5 135.3 45) (layer "Cmts.User")
     (effects (font (size 1 1) (thickness 0.154)) (justify left bottom))
   )
@@
   )
   (dimension (type aligned) (layer "Dwgs.User")
-    (pts (xy 119.38 129.54) (xy 165.1 129.54))
+    (pts (xy 119.38 136.02) (xy 165.1 136.02))
     (height 5.08)
-    (gr_text "45.7200 mm" (at 142.24 133.466) (layer "Dwgs.User")
+    (gr_text "45.7200 mm" (at 142.24 139.946) (layer "Dwgs.User")
       (effects (font (size 1 1) (thickness 0.154)))
     )
@@
   )
   (dimension (type aligned) (layer "Dwgs.User")
-    (pts (xy 117.212 128.15) (xy 166.488 128.15))
+    (pts (xy 117.212 134.63) (xy 166.488 134.63))
     (height 9.7)
-    (gr_text "49.2760 mm" (at 141.85 136.696) (layer "Dwgs.User")
+    (gr_text "49.2760 mm" (at 141.85 143.176) (layer "Dwgs.User")
       (effects (font (size 1 1) (thickness 0.154)))
     )
