File: circuits/OSSI_CM2V2.0/OSSI_CM2.kicad_sch (KiCad schematic)
At the start: 80 parts, among them U101 STM32L412C8T6, U102 M24M01, U103 LM75B, U104 OPA2317, X101 PINHEADER_2×5, X201 Conn_01x20_Pin, X202 Conn_01x21_Pin, Y101 10MHz

Commit message: cleans up routing, library links, library 3D models
Parts:
- C101, C102, C103, C104, C105, C106, C107, C108, C109, C110, C111, C112, C113, C115, C116, C117, C119, C120, C122, C125, C126: footprint OSSI_standard_footprints:0603_W -> OSSI_standard_footprints:0603_W_C
- C114, C118, C121, C123, C124: footprint OSSI_standard_footprints:0805_W -> OSSI_standard_footprints:0805_W_C
- H140: value LED -> LED gn
- H141: value LED -> LED rd
- L101: footprint OSSI_standard_footprints:0805_W -> OSSI_standard_footprints:0805_W_L
- R101, R102, R103, R104, R105, R106, R107, R108, R109, R110, R111, R112, R113, R114, R115, R116, R117, R118, R119, R120, R121, R122, R123, R124, R125, R126, R127, R128, R129, R130, R131, R132, R133, R134, R135, R136, R137, R140, R141: footprint OSSI_standard_footprints:0603_W -> OSSI_standard_footprints:0603_W_R
