File: circuits/OSSI_CM2V2.0/OSSI_CM2.kicad_sch (KiCad schematic)
At the start: 80 parts, among them U101 STM32L412C8T6, U102 M24M01, U103 LM75B, U104 OPA2317, X101 PINHEADER_2×5, X201 Conn_01x20_Pin, X202 Conn_01x21_Pin, Y101 10MHz

Commit message: cleans up and rearranges schematics for more clarity
Parts:
- D101: Manufacturer Texas Instruments -> M
Connections:
- net BOOT: now reaches BOOT0.2, R131.2, U101.44 (PH3/BOOT0), X101.8
- net ~{RESET}: now reaches R136.2, RESET0.2, U101.7 (~{RST}), X101.10
Other:
- note added: "Input to Module"
- note added: "Output from Module"
- moved on the sheet: BOOT0, C103, C104, C105, C106, C107, C109, C110, C112, C115, C116, C117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
